File: Test_board/power_schematic.sch (KiCad schematic (older format))
At the start: 65 parts, among them J10 4.19mmBananaJack, J13 4.19mmBananaJack, J14 4.19mmBananaJack, J9 4.19mmBananaJack, U3 LT3652, U5 LT3652, U6 TPS63000, U7 LM193, U8 TPS22965-Q1, U9 TPS22965-Q1

Commit message: Replaced TPS63000 with new IC and started wiring it. Started migrating previous libraries to new global Aleksandr library.
Parts:
- removed C27, C28: 22uF, Capacitors_SMD:C_0805, symbol C
- removed J13, J14: 4.19mmBananaJack, aleksandr_footprints:4.19Banana, symbol 4.19mmBananaJack
- removed L3: 1.5uH, aleksandr_footprints:SMD-1008, symbol L
- removed R33: 1M, Resistors_SMD:R_0805, symbol R
- removed R34: 178k, Resistors_SMD:R_0805, symbol R
- removed U6: TPS63000, Housings_DFN_QFN:DFN-10-1EP_3x3mm_Pitch0.5mm, symbol TPS63000
- added C?: C, symbol C
- added J?: USB_OTG, symbol USB_OTG
- added J? (x2): 4.19mmBananaJack, symbol 4.19mmBananaJack
- added L?: L, symbol L
- added R? (x2): R, symbol R
- added U?: S6BP203A, symbol S6BP203A
Connections:
- wire segments 163 -> 171
- no-connect marks 8 -> 11
