File: Test_board/Test_board.kicad_pcb (KiCad board)
At the start: 4 copper layers, 94 x 94 mm, 131 parts, among them J1 CONN_02X26, J10 4.19mmBananaJack, J11 4.19mmBananaJack, J12 4.19mmBananaJack, J13 4.19mmBananaJack, J14 USB_OTG, J15 TEST_1P, J16 TEST_1P, J17 Conn_01x02, J18 TEST_1P, J2 CONN_02X26, J3 Conn_02x05_Odd_Even, J4 Conn_01x03, J5 Conn_02x20_Odd_Even, J7 Conn_01x06, J8 Conn_02x20_Odd_Even, J9 USB_A, Q1 Q_NMOS_GSD, U1 STM32F303RE, U10 INA219, U11 INA219, U12 MS5540C, U2 24LC256, U3 LT3652, U4 INA219, U5 LTC3113, U6 MAX6730A, U7 LTC3113, U8 LT3652, U9 INA219

Commit message: finished pcb
Parts:
- removed C10, C25 (x2): 100uF, Capacitors_SMD:C_0805_HandSoldering
- removed C11: 47uF, Capacitors_SMD:C_0805_HandSoldering
- removed C17 (x2): 0.1uF, Capacitors_SMD:C_0805_HandSoldering
- removed C19 (x2): 1uF, Capacitors_SMD:C_0805_HandSoldering
- removed C23 (x2): 10uF, Capacitors_SMD:C_0805_HandSoldering
- removed C27: 12pF, Capacitors_SMD:C_0805_HandSoldering
- removed C29: 680pF, Capacitors_SMD:C_0805_HandSoldering
- removed C31: 47pF, Capacitors_SMD:C_0805_HandSoldering
- removed D2 (x2): MBRS140, Diodes_SMD:D_SMB
- removed D4 (x2): MBRS340, Diodes_SMD:D_SMC
- removed D6 (x2): D, aleksandr_footprints:SOD-123FL
- removed J15: TEST_1P, Measurement_Points:Measurement_Point_Round-SMD-Pad_Big
- removed J9: USB_A, aleksandr_footprints:USB_A_Board
- removed L1: 2.2uH, aleksandr_footprints:L-7443330220
- removed L4 (x2): 6.8uH, aleksandr_footprints:L-SLF6028T-6R8M1R5-PF
- removed R16 (x2), R17 (x2), R18 (x2): 100k, Resistors_SMD:R_0805_HandSoldering
- removed R20 (x2): 179k, Resistors_SMD:R_0805_HandSoldering
- removed R22 (x2): 330k, Resistors_SMD:R_0805_HandSoldering
- removed R25 (x2), R26 (x2): 180k, Resistors_SMD:R_0805_HandSoldering
- removed R28 (x2): 50m, Resistors_SMD:R_1206_HandSoldering
- removed R30: 49.9k, Resistors_SMD:R_0805_HandSoldering
- removed R31: 887k, Resistors_SMD:R_0805_HandSoldering
- removed R32: 121k, Resistors_SMD:R_0805_HandSoldering
- removed R34: 6.49k, Resistors_SMD:R_0805_HandSoldering
- removed R7: 90.9k, Resistors_SMD:R_0805_HandSoldering
- removed U5: LTC3113, aleksandr_footprints:20TSSOP-E
- removed U8 (x2): LT3652, aleksandr_footprints:12MSOP-E
- added C33: 0.1uF, Capacitors_SMD:C_0805_HandSoldering, B.Cu at (169.8, 40.4)
- C1, C14, C15, C2, C20, C21, C3, C4, R9, U1, U10, U11, U4, U9: moved to B.Cu
- moved J14 218.4 mm to (192.3, 29.3), turned to 180 degrees
- moved C21 192.2 mm to (203.3, 58.9), turned to 270 degrees
- moved U4 190.0 mm to (188.6, 55.6)
- moved J12 189.2 mm to (201.8, 32.6), turned to 90 degrees
- moved C12 185.6 mm to (200.8, 60.3)
- moved R29 180.6 mm to (203.3, 72.6), turned to 270 degrees
- moved J13 178.2 mm to (212.0, 32.6), turned to 90 degrees
- moved C30 177.3 mm to (199.3, 72.6), turned to 270 degrees
- moved C15 176.9 mm to (190.1, 52.0)
- moved R12 173.7 mm to (197.7, 75.9), turned to 180 degrees
- moved C26 169.3 mm to (202.3, 75.9)
- moved R3 167.2 mm to (179.7, 41.4)
- moved C13 166.8 mm to (195.1, 66.0), turned to 270 degrees
- moved R33 166.0 mm to (195.7, 71.7)
- moved C28 165.5 mm to (201.3, 72.6), turned to 90 degrees
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Connections:
- net /USB_D+ renamed Net-(J8-Pad21)
- net /USB_D- renamed Net-(J8-Pad19)
- J12 pad 1: /POWER/VINPUT -> +BATT
- J14 pad 1: /POWER/VINPUT -> +BATT
- U1 pad 16: /ARM_UART2_MISO -> /L_MCU_GND
- U1 pad 17: /ARM_UART2_MOSI -> /L_MCU_GND
- U1 pad 21: /ARM_SPI1_SCK -> /B_MCU_GND
- U1 pad 22: /ARM_SPI1_MISO -> /B_MCU_GND
- U1 pad 23: /ARM_SPI1_MOSI -> /B_MCU_GND
- U1 pad 25: (no net) -> /UART0_MOSI
- U1 pad 26: /UART0_MOSI -> /B_MCU_GND
- U1 pad 44: /ARM_USB_D- -> /B_MCU_GND
- U1 pad 45: /ARM_USB_D+ -> /B_MCU_GND
- U1 pad 61: /CAN_RX -> /T_MCU_GND
- U1 pad 62: /CAN_TX -> /T_MCU_GND
Routing:
- net /SDA0: track 6.35 -> 230.3 mm, vias 0 -> 12
- net /SCL0: track 6.35 -> 222.5 mm, vias 0 -> 7
- net +BATT: track 0.00 -> 181.9 mm, vias 0 -> 5
- net GND: track 152.0 -> 264.5 mm, vias 24 -> 76
- net Net-(J8-Pad19): track 77.5 -> 6.35 mm, vias 1 -> 0
- net Net-(J8-Pad21): track 76.0 -> 6.35 mm, vias 1 -> 0
- net +3V3: track 18.3 -> 86.7 mm, vias 6 -> 24
- net /POWER/VOUT3: track 0.00 -> 46.7 mm, vias 0 -> 2
- net /UART0_MOSI: track 26.7 -> 71.9 mm, vias 0 -> 1
- net /UART0_MISO: track 6.35 -> 43.8 mm, vias 0 -> 1
- net /ARM_MSTR_RST: track 26.7 -> 59.0 mm, vias 0 -> 1
- net /EEPROM_WP: track 27.7 -> 55.4 mm, vias 0 -> 1
- net /ARM_RST: track 0.00 -> 22.8 mm, vias 0 -> 4
- net Net-(L2-Pad2): track 0.00 -> 21.8 mm
- net Net-(C26-Pad1): track 0.00 -> 21.2 mm, vias 0 -> 2
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Other:
- net class Default: clearance 0.381 -> 0.1524
- net class Tight added: clearance 0.127, trace_width 0.508, via_dia 0.6, via_drill 0.4
- rule trace_clearance: 0.381 -> 0.1524
- rule via_min_drill: 0.254 -> 0.3
