File: Test_board/power.sch (KiCad schematic (older format))
At the start: 75 parts, among them J10 4.19mmBananaJack, J11 4.19mmBananaJack, J12 4.19mmBananaJack, J13 4.19mmBananaJack, J14 USB_OTG, J15 TEST_1P, J16 TEST_1P, U10 INA219, U11 INA219, U3 LT3652, U4 INA219, U5 LTC3113, U7 LTC3113, U8 LT3652, U9 INA219

Commit message: Removed db9, created last footprints, finished assigning footprints, started pcb
Parts:
- D5, D6: footprint (none) -> aleksandr_footprints:SOD-123FL
- J14: footprint (none) -> aleksandr_footprints:micro_usb_smd
Changed lines of the file:
@@
 Sheet 2 2
 Title "ARIETTA TEST BOARD"
-Date ""
+Date "2017-11-08"
 Rev "2"
 Comp ""
 Comment1 "D. FERNIE"
-Comment2 ""
+Comment2 "D. FERNIE"
 Comment3 ""
 Comment4 ""
@@
 F 0 "J14" H 800 2550 50  0000 L CNN
 F 1 "USB_OTG" H 800 2450 50  0000 L CNN
-F 2 "" H 1150 2050 50  0001 C CNN
+F 2 "aleksandr_footprints:micro_usb_smd" H 1150 2050 50  0001 C CNN
 F 3 "" H 1150 2050 50  0001 C CNN
 	1    1000 2100
@@
 VIN
 $Comp
-L GND #PWR045
+L GND #PWR044
 U 1 1 59FD2EC2
 P 1200 3000
-F 0 "#PWR045" H 1200 2750 50  0001 C CNN
+F 0 "#PWR044" H 1200 2750 50  0001 C CNN
 F 1 "GND" H 1200 2850 50  0000 C CNN
 F 2 "" H 1200 3000 50  0001 C CNN
@@
 $EndComp
 $Comp
-L GND #PWR046
+L GND #PWR045
 U 1 1 59FFAE5F
 P 10000 2100
-F 0 "#PWR046" H 10000 1850 50  0001 C CNN
+F 0 "#PWR045" H 10000 1850 50  0001 C CNN
 F 1 "GND" H 10000 1950 50  0000 C CNN
 F 2 "" H 10000 2100 50  0001 C CNN
@@
 $EndComp
 $Comp
-L GND #PWR047
+L GND #PWR046
 U 1 1 59FFB67F
 P 9500 3850
-F 0 "#PWR047" H 9500 3600 50  0001 C CNN
+F 0 "#PWR046" H 9500 3600 50  0001 C CNN
 F 1 "GND" H 9500 3700 50  0000 C CNN
 F 2 "" H 9500 3850 50  0001 C CNN
@@
 SDA
 $Comp
-L +3V3 #PWR048
+L +3V3 #PWR047
 U 1 1 59FFFEC7
 P 2300 5050
-F 0 "#PWR048" H 2300 4900 50  0001 C CNN
+F 0 "#PWR047" H 2300 4900 50  0001 C CNN
 F 1 "+3V3" H 2300 5190 50  0000 C CNN
 F 2 "" H 2300 5050 50  0001 C CNN
@@
 $EndComp
 $Comp
-L +3V3 #PWR049
+L +3V3 #PWR048
 U 1 1 59FFFF81
 P 4750 5050
-F 0 "#PWR049" H 4750 4900 50  0001 C CNN
+F 0 "#PWR048" H 4750 4900 50  0001 C CNN
 F 1 "+3V3" H 4750 5190 50  0000 C CNN
 F 2 "" H 4750 5050 50  0001 C CNN
@@
 $EndComp
 $Comp
-L GND #PWR050
+L GND #PWR049
 U 1 1 5A0000B7
 P 2450 4950
-F 0 "#PWR050" H 2450 4700 50  0001 C CNN
+F 0 "#PWR049" H 2450 4700 50  0001 C CNN
 F 1 "GND" H 2450 4800 50  0000 C CNN
 F 2 "" H 2450 4950 50  0001 C CNN
@@
 $EndComp
 $Comp
-L GND #PWR051
+L GND #PWR050
 U 1 1 5A0001CD
 P 4900 4950
-F 0 "#PWR051" H 4900 4700 50  0001 C CNN
+F 0 "#PWR050" H 4900 4700 50  0001 C CNN
 F 1 "GND" H 4900 4800 50  0000 C CNN
 F 2 "" H 4900 4950 50  0001 C CNN
@@
 	1300 4750 1300 4850
 $Comp
-L GND #PWR052
+L GND #PWR051
 U 1 1 5A0012AA
 P 1250 4750
-F 0 "#PWR052" H 1250 4500 50  0001 C CNN
+F 0 "#PWR051" H 1250 4500 50  0001 C CNN
 F 1 "GND" H 1250 4600 50  0000 C CNN
 F 2 "" H 1250 4750 50  0001 C CNN
@@
 Connection ~ 1300 4750
 $Comp
-L GND #PWR053
+L GND #PWR052
 U 1 1 5A0013A5
 P 3700 4750
-F 0 "#PWR053" H 3700 4500 50  0001 C CNN
+F 0 "#PWR052" H 3700 4500 50  0001 C CNN
 F 1 "GND" H 3700 4600 50  0000 C CNN
 F 2 "" H 3700 4750 50  0001 C CNN
@@
 	3700 4750 3750 4750
 $Comp
-L +3V3 #PWR054
+L +3V3 #PWR053
 U 1 1 5A0014A0
 P 3600 4850
-F 0 "#PWR054" H 3600 4700 50  0001 C CNN
+F 0 "#PWR053" H 3600 4700 50  0001 C CNN
 F 1 "+3V3" H 3600 4990 50  0000 C CNN
 F 2 "" H 3600 4850 50  0001 C CNN
@@
 F 0 "D5" H 4900 1100 50  0000 C CNN
 F 1 "D" H 4900 900 50  0000 C CNN
-F 2 "" H 4900 1000 50  0001 C CNN
+F 2 "aleksandr_footprints:SOD-123FL" H 4900 1000 50  0001 C CNN
 F 3 "" H 4900 1000 50  0001 C CNN
 	1    4900 1000
@@
 Connection ~ 5250 1000
 $Comp
-L GND #PWR055
+L GND #PWR054
 U 1 1 5A014DF0
 P 4050 650
-F 0 "#PWR055" H 4050 400 50  0001 C CNN
+F 0 "#PWR054" H 4050 400 50  0001 C CNN
 F 1 "GND" H 4050 500 50  0000 C CNN
 F 2 "" H 4050 650 50  0001 C CNN
@@
 Connection ~ 5450 700
 $Comp
-L GND #PWR056
+L GND #PWR055
 U 1 1 5A015772
 P 3850 2000
-F 0 "#PWR056" H 3850 1750 50  0001 C CNN
+F 0 "#PWR055" H 3850 1750 50  0001 C CNN
 F 1 "GND" H 3850 1850 50  0000 C CNN
 F 2 "" H 3850 2000 50  0001 C CNN
@@
 F 0 "D6" H 4900 2750 50  0000 C CNN
 F 1 "D" H 4900 2550 50  0000 C CNN
-F 2 "" H 4900 2650 50  0001 C CNN
+F 2 "aleksandr_footprints:SOD-123FL" H 4900 2650 50  0001 C CNN
 F 3 "" H 4900 2650 50  0001 C CNN
 	1    4900 2650
@@
 Connection ~ 5250 2650
 $Comp
-L GND #PWR057
+L GND #PWR056
 U 1 1 5A016254
 P 4050 2300
-F 0 "#PWR057" H 4050 2050 50  0001 C CNN
+F 0 "#PWR056" H 4050 2050 50  0001 C CNN
 F 1 "GND" H 4050 2150 50  0000 C CNN
 F 2 "" H 4050 2300 50  0001 C CNN
@@
 Connection ~ 5450 2350
 $Comp
-L GND #PWR058
+L GND #PWR057
 U 1 1 5A016262
 P 3850 3650
-F 0 "#PWR058" H 3850 3400 50  0001 C CNN
+F 0 "#PWR057" H 3850 3400 50  0001 C CNN
 F 1 "GND" H 3850 3500 50  0000 C CNN
 F 2 "" H 3850 3650 50  0001 C CNN
@@
 Connection ~ 2150 5050
 $Comp
-L GND #PWR059
+L GND #PWR058
 U 1 1 5A01C939
 P 2150 5450
-F 0 "#PWR059" H 2150 5200 50  0001 C CNN
+F 0 "#PWR058" H 2150 5200 50  0001 C CNN
 F 1 "GND" H 2150 5300 50  0000 C CNN
 F 2 "" H 2150 5450 50  0001 C CNN
@@
 Connection ~ 4600 5050
 $Comp
-L GND #PWR060
+L GND #PWR059
 U 1 1 5A01D246
 P 4600 5450
-F 0 "#PWR060" H 4600 5200 50  0001 C CNN
+F 0 "#PWR059" H 4600 5200 50  0001 C CNN
 F 1 "GND" H 4600 5300 50  0000 C CNN
 F 2 "" H 4600 5450 50  0001 C CNN
@@
 SDA
 $Comp
-L +3V3 #PWR061
+L +3V3 #PWR060
 U 1 1 5A01D951
 P 2300 6650
-F 0 "#PWR061" H 2300 6500 50  0001 C CNN
+F 0 "#PWR060" H 2300 6500 50  0001 C CNN
 F 1 "+3V3" H 2300 6790 50  0000 C CNN
 F 2 "" H 2300 6650 50  0001 C CNN
@@
 $EndComp
 $Comp
-L +3V3 #PWR062
+L +3V3 #PWR061
 U 1 1 5A01D957
 P 4750 6650
-F 0 "#PWR062" H 4750 6500 50  0001 C CNN
+F 0 "#PWR061" H 4750 6500 50  0001 C CNN
 F 1 "+3V3" H 4750 6790 50  0000 C CNN
 F 2 "" H 4750 6650 50  0001 C CNN
@@
 $EndComp
 $Comp
-L GND #PWR063
+L GND #PWR062
 U 1 1 5A01D95D
 P 2450 6550
-F 0 "#PWR063" H 2450 6300 50  0001 C CNN
+F 0 "#PWR062" H 2450 6300 50  0001 C CNN
 F 1 "GND" H 2450 6400 50  0000 C CNN
 F 2 "" H 2450 6550 50  0001 C CNN
@@
 $EndComp
 $Comp
-L GND #PWR064
+L GND #PWR063
 U 1 1 5A01D963
 P 4900 6550
-F 0 "#PWR064" H 4900 6300 50  0001 C CNN
+F 0 "#PWR063" H 4900 6300 50  0001 C CNN
 F 1 "GND" H 4900 6400 50  0000 C CNN
 F 2 "" H 4900 6550 50  0001 C CNN
@@
 	1300 6350 1300 6450
 $Comp
-L GND #PWR065
+L GND #PWR064
 U 1 1 5A01D96C
 P 1250 6350
-F 0 "#PWR065" H 1250 6100 50  0001 C CNN
+F 0 "#PWR064" H 1250 6100 50  0001 C CNN
 F 1 "GND" H 1250 6200 50  0000 C CNN
 F 2 "" H 1250 6350 50  0001 C CNN
@@
 Connection ~ 1300 6350
 $Comp
-L GND #PWR066
+L GND #PWR065
 U 1 1 5A01D974
 P 3700 6350
-F 0 "#PWR066" H 3700 6100 50  0001 C CNN
+F 0 "#PWR065" H 3700 6100 50  0001 C CNN
 F 1 "GND" H 3700 6200 50  0000 C CNN
 F 2 "" H 3700 6350 50  0001 C CNN
@@
 	3700 6350 3750 6350
 $Comp
-L +3V3 #PWR067
+L +3V3 #PWR066
 U 1 1 5A01D97B
 P 3600 6450
-F 0 "#PWR067" H 3600 6300 50  0001 C CNN
+F 0 "#PWR066" H 3600 6300 50  0001 C CNN
 F 1 "+3V3" H 3600 6590 50  0000 C CNN
 F 2 "" H 3600 6450 50  0001 C CNN
@@
 Connection ~ 2150 6650
 $Comp
-L GND #PWR068
+L GND #PWR067
 U 1 1 5A01D9A1
 P 2150 7050
-F 0 "#PWR068" H 2150 6800 50  0001 C CNN
+F 0 "#PWR067" H 2150 6800 50  0001 C CNN
 F 1 "GND" H 2150 6900 50  0000 C CNN
 F 2 "" H 2150 7050 50  0001 C CNN
@@
 Connection ~ 4600 6650
 $Comp
-L GND #PWR069
+L GND #PWR068
 U 1 1 5A01D9B0
 P 4600 7050
-F 0 "#PWR069" H 4600 6800 50  0001 C CNN
+F 0 "#PWR068" H 4600 6800 50  0001 C CNN
 F 1 "GND" H 4600 6900 50  0000 C CNN
 F 2 "" H 4600 7050 50  0001 C CNN
@@
 VOUT3
 $Comp
-L +3V3 #PWR070
+L +3V3 #PWR069
 U 1 1 5A01FE6F
 P 2750 6600
-F 0 "#PWR070" H 2750 6450 50  0001 C CNN
+F 0 "#PWR069" H 2750 6450 50  0001 C CNN
 F 1 "+3V3" H 2750 6740 50  0000 C CNN
 F 2 "" H 2750 6600 50  0001 C CNN
@@
 3V3 bus monitoring
 $Comp
-L +5V #PWR071
+L +5V #PWR070
 U 1 1 5A022D0F
 P 10950 2900
-F 0 "#PWR071" H 10950 2750 50  0001 C CNN
+F 0 "#PWR070" H 10950 2750 50  0001 C CNN
 F 1 "+5V" H 10950 3040 50  0000 C CNN
 F 2 "" H 10950 2900 50  0001 C CNN
@@
 Connection ~ 10950 2950
 $Comp
-L +BATT #PWR072
+L +BATT #PWR071
 U 1 1 5A023886
 P 2850 5000
-F 0 "#PWR072" H 2850 4850 50  0001 C CNN
+F 0 "#PWR071" H 2850 4850 50  0001 C CNN
 F 1 "+BATT" H 2850 5140 50  0000 C CNN
 F 2 "" H 2850 5000 50  0001 C CNN
@@
 Connection ~ 2850 4950
 $Comp
-L GND #PWR073
+L GND #PWR072
 U 1 1 5A02AE9E
 P 8950 2400
-F 0 "#PWR073" H 8950 2150 50  0001 C CNN
+F 0 "#PWR072" H 8950 2150 50  0001 C CNN
 F 1 "GND" H 8950 2250 50  0000 C CNN
 F 2 "" H 8950 2400 50  0001 C CNN
@@
 Connection ~ 9000 2400
 $Comp
-L GND #PWR074
+L GND #PWR073
 U 1 1 5A02B7BE
 P 8950 500
-F 0 "#PWR074" H 8950 250 50  0001 C CNN
+F 0 "#PWR073" H 8950 250 50  0001 C CNN
 F 1 "GND" H 8950 350 50  0000 C CNN
 F 2 "" H 8950 500 50  0001 C CNN

Commit message: finished pcb
Parts:
- removed C10, C25: 100uF, Capacitors_SMD:C_0805_HandSoldering, symbol C
- removed C11: 47uF, Capacitors_SMD:C_0805_HandSoldering, symbol C
- removed C17: 0.1uF, Capacitors_SMD:C_0805_HandSoldering, symbol C
- removed C19: 1uF, Capacitors_SMD:C_0805_HandSoldering, symbol C
- removed C23: 10uF, Capacitors_SMD:C_0805_HandSoldering, symbol C
- removed C27: 12pF, Capacitors_SMD:C_0805_HandSoldering, symbol C
- removed C29: 680pF, Capacitors_SMD:C_0805_HandSoldering, symbol C
- removed C31: 47pF, Capacitors_SMD:C_0805_HandSoldering, symbol C
- removed D2: MBRS140, Diodes_SMD:D_SMB, symbol D_Schottky
- removed D4: MBRS340, Diodes_SMD:D_SMC, symbol D_Schottky
- removed D6: D, aleksandr_footprints:SOD-123FL, symbol D
- removed J15: TEST_1P, Measurement_Points:Measurement_Point_Round-SMD-Pad_Big, symbol TEST_1P
- removed L1: 2.2uH, aleksandr_footprints:L-7443330220, symbol L
- removed L4: 6.8uH, aleksandr_footprints:L-SLF6028T-6R8M1R5-PF, symbol L
- removed R16, R17, R18: 100k, Resistors_SMD:R_0805_HandSoldering, symbol R
- removed R20: 179k, Resistors_SMD:R_0805_HandSoldering, symbol R
- removed R22: 330k, Resistors_SMD:R_0805_HandSoldering, symbol R
- removed R25, R26: 180k, Resistors_SMD:R_0805_HandSoldering, symbol R
- removed R28: 50m, Resistors_SMD:R_1206_HandSoldering, symbol R
- removed R30: 49.9k, Resistors_SMD:R_0805_HandSoldering, symbol R
- removed R31: 887k, Resistors_SMD:R_0805_HandSoldering, symbol R
- removed R32: 121k, Resistors_SMD:R_0805_HandSoldering, symbol R
- removed R34: 6.49k, Resistors_SMD:R_0805_HandSoldering, symbol R
- removed R7: 90.9k, Resistors_SMD:R_0805_HandSoldering, symbol R
- removed U5: LTC3113, aleksandr_footprints:20TSSOP-E, symbol LTC3113
- removed U8: LT3652, aleksandr_footprints:12MSOP-E, symbol LT3652
Connections:
- net VINPUT is gone; now on net +BATT: J12.1, J14.1 (VBUS)
- no-connect marks 9 -> 6
Other:
- note removed: "5V"
