File: Test_board/test_board.sch (KiCad schematic (older format))
At the start: 31 parts, among them J1 CONN_02X26, J2 CONN_02X26, J3 Conn_02x05_Odd_Even, J4 Conn_01x03, J5 Conn_02x20_Odd_Even, J6 DB9_Male, J7 Conn_01x06, J8 Conn_02x20_Odd_Even, J9 USB_A, U1 STM32F303RE, U2 24LC256

Commit message: Finished schematic
Parts:
- added C32, C9: 0.1uF, Capacitors_SMD:C_0805_HandSoldering, symbol C
- added J17: Conn_01x02, Pin_Headers:Pin_Header_Straight_1x02_Pitch2.54mm, symbol Conn_01x02
- added J18: TEST_1P, Measurement_Points:Measurement_Point_Round-SMD-Pad_Big, symbol TEST_1P
- added U12: MS5540C, symbol MS5540C
- C1, C2, C3, C4, C5, C6, C7, C8: footprint 0805 -> Capacitors_SMD:C_0805_HandSoldering
- J3: footprint (none) -> Pin_Headers:Pin_Header_Straight_2x05_Pitch2.54mm
- J4: footprint (none) -> Pin_Headers:Pin_Header_Straight_1x03_Pitch2.54mm
- J5, J8: footprint (none) -> Pin_Headers:Pin_Header_Straight_2x20_Pitch2.54mm
- J7: footprint (none) -> Pin_Headers:Pin_Header_Straight_1x06_Pitch2.54mm
- R1, R2, R3, R4: footprint 0805 -> (none)
- R5, R6: renamed from R?; footprint 0805 -> (none)
- gave numbers to parts that had none: 2
Connections:
- net +3V3: now also C1.1, C2.1, C3.1, C4.1, C5.1, SN1.4 (VCC), SN1.6 (~RST), U1.13 (VDDA), U1.19 (VDD), U1.32 (VDD), U1.48 (VDD), U1.64 (VDD), C32.1, J17.1 (Pin_1), U12.5 (VDD); no longer U6.4 (~MR), U6.6 (VCC)
- net B_MCU_GND: no longer U1.21 (PA5), U1.22 (PA6), U1.23 (PA7), U1.44 (PA11), U1.45 (PA12)
- net GND: now also C1.2, C2.2, C3.2, C4.2, C5.2, J1.18 (P18), J1.20 (P20), J1.22 (P22), J1.24 (P24), J1.26 (P26), J1.28 (P28), J1.30 (P30), J1.31 (P31), J1.32 (P32), J1.34 (P34), J1.36 (P36), J1.37 (P37), J1.38 (P38), Q1.2 (S), SN1.10 (NC), SN1.11 (NC), SN1.12 (NC), SN1.13 (NC), SN1.14 (NC), SN1.15 (GND), SN1.16 (VBAT), SN1.7 (NC), SN1.8 (NC), SN1.9 (NC), U1.1 (VBAT), U1.12 (GNDA), U1.18 (GND), U1.31 (GND), U1.47 (GND), U1.63 (GND), C32.2, C9.2, U12.2 (GND)
- net L_MCU_GND: no longer U1.16 (PA2), U1.17 (PA3)
- net T_MCU_GND: no longer U1.61 (PB8), U1.62 (PB9)
- net WDT_KICK: now also J5.31 (Pin_31), J5.32 (Pin_32), OBC1.31 (PC4); no longer J5.15 (Pin_15), J5.16 (Pin_16), OBC1.15 (PA26)
- net ARM_SPI1_SCK: now reaches J1.17 (P17)
- net ARM_SPI1_SCK: now also U1.21 (PA5)
- net ARM_SPI1_MISO: now reaches J1.19 (P19)
- net ARM_SPI1_MISO: now also U1.22 (PA6)
- net ARM_SPI1_MOSI: now reaches J1.21 (P21)
- net ARM_SPI1_MOSI: now also U1.23 (PA7)
- net ARM_UART2_MISO: now reaches J1.23 (P23)
- net ARM_UART2_MISO: now also U1.16 (PA2)
- net ARM_UART2_MOSI: now reaches J1.25 (P25)
- net ARM_UART2_MOSI: now also U1.17 (PA3)
- net ARM_USB_D-: now reaches J1.27 (P27)
- net ARM_USB_D-: now also U1.44 (PA11)
- net ARM_USB_D+: now reaches J1.29 (P29)
- net ARM_USB_D+: now also U1.45 (PA12)
- net CAN_RX: now reaches J1.33 (P33)
- net CAN_RX: now also U1.61 (PB8)
- net CAN_TX: now reaches J1.35 (P35)
- net CAN_TX: now also U1.62 (PB9)
- net BARO_CLK: now reaches J5.11 (Pin_11), J5.12 (Pin_12), OBC1.11 (PA24)
- net BARO_CLK: now also U12.1 (SCLK)
- net BARO_MISO: now reaches J5.13 (Pin_13), J5.14 (Pin_14), OBC1.13 (PA25)
- net BARO_MISO: now also U12.8 (DOUT)
- net 32kHz: now reaches SN1.3 (32kHz)
- net 32kHz: now also J18.1, U12.6 (MCLK)
- net at U6.3 (~WDO): now also U6.4 (~MR)
- net ARM_SWIM: no longer names the net of J3.3 (Pin_3)
- new net: C9.1, J17.2 (Pin_2), U6.6 (VCC)
- new net BARO_MOSI: J5.15 (Pin_15), J5.16 (Pin_16), OBC1.15 (PA26), U12.7 (DIN)
- no-connect marks 73 -> 50
Other:
- note added: "Barometer"

Commit message: Updated libraries, footprint assignments, and created protector for barometer
Parts:
- J9: footprint (none) -> aleksandr_footprints:USB_A_Board
- OBC1: footprint (none) -> aleksandr_footprints:Arietta_G25
- Q1: footprint (none) -> TO_SOT_Packages_SMD:SOT-23_Handsoldering
- R1, R2, R3, R4, R5, R6: footprint (none) -> Resistors_SMD:R_0805_HandSoldering
- SN1: footprint (none) -> Housings_SOIC:SOIC-20W_7.5x12.8mm_Pitch1.27mm
- SN2, SN3: footprint (none) -> Housings_SOIC:SOIJ-8_5.3x5.3mm_Pitch1.27mm
- U1: footprint (none) -> Housings_QFP:LQFP-64_10x10mm_Pitch0.5mm
- U12: footprint (none) -> aleksandr_footprints:MS5540C
- U2: footprint Housings_SOIC:SOIC-8_3.9x4.9mm_Pitch1.27mm -> Housings_DIP:DIP-8_W7.62mm_Socket
- U6: footprint (none) -> TO_SOT_Packages_SMD:SOT-23-6_Handsoldering
Changed lines of the file:
@@
 F 0 "OBC1" H 7000 3800 60  0000 C CNN
 F 1 "Arietta_G25" H 7000 5900 60  0000 C CNN
-F 2 "" H 7000 4800 60  0001 C CNN
+F 2 "aleksandr_footprints:Arietta_G25" H 7000 4800 60  0001 C CNN
 F 3 "" H 7000 4800 60  0001 C CNN
 	1    7000 4800
@@
 F 0 "J9" H 7850 3450 50  0000 L CNN
 F 1 "USB_A" H 7850 3350 50  0000 L CNN
-F 2 "" H 8200 2950 50  0001 C CNN
+F 2 "aleksandr_footprints:USB_A_Board" H 8200 2950 50  0001 C CNN
 F 3 "" H 8200 2950 50  0001 C CNN
 	1    8050 3000
@@
 F 0 "U1" H 3250 4000 60  0000 C CNN
 F 1 "STM32F303RE" H 3250 7700 60  0000 C CNN
-F 2 "" H 3250 5750 60  0001 C CNN
+F 2 "Housings_QFP:LQFP-64_10x10mm_Pitch0.5mm" H 3250 5750 60  0001 C CNN
 F 3 "" H 3250 5750 60  0001 C CNN
 	1    3250 5750
@@
 F 0 "R4" V 2130 3850 50  0000 C CNN
 F 1 "4K7" V 2050 3850 50  0000 C CNN
-F 2 "" V 1980 3850 50  0001 C CNN
+F 2 "Resistors_SMD:R_0805_HandSoldering" V 1980 3850 50  0001 C CNN
 F 3 "" H 2050 3850 50  0001 C CNN
 	1    2050 3850
@@
 F 0 "R1" V 830 7200 50  0000 C CNN
 F 1 "4k7" V 750 7200 50  0000 C CNN
-F 2 "" V 680 7200 50  0001 C CNN
+F 2 "Resistors_SMD:R_0805_HandSoldering" V 680 7200 50  0001 C CNN
 F 3 "" H 750 7200 50  0001 C CNN
 	1    750  7200
@@
 F 0 "R2" V 1080 7200 50  0000 C CNN
 F 1 "4k7" V 1000 7200 50  0000 C CNN
-F 2 "" V 930 7200 50  0001 C CNN
+F 2 "Resistors_SMD:R_0805_HandSoldering" V 930 7200 50  0001 C CNN
 F 3 "" H 1000 7200 50  0001 C CNN
 	1    1000 7200
@@
 F 0 "R3" V 1330 7200 50  0000 C CNN
 F 1 "4k7" V 1250 7200 50  0000 C CNN
-F 2 "" V 1180 7200 50  0001 C CNN
+F 2 "Resistors_SMD:R_0805_HandSoldering" V 1180 7200 50  0001 C CNN
 F 3 "" H 1250 7200 50  0001 C CNN
 	1    1250 7200
@@
 F 0 "SN2" H 8050 600 60  0000 C CNN
 F 1 "DS1624" H 8050 1200 60  0000 C CNN
-F 2 "" H 8050 900 60  0001 C CNN
+F 2 "Housings_SOIC:SOIJ-8_5.3x5.3mm_Pitch1.27mm" H 8050 900 60  0001 C CNN
 F 3 "" H 8050 900 60  0001 C CNN
 	1    8050 900
@@
 F 0 "SN3" H 8050 1350 60  0000 C CNN
 F 1 "DS1624" H 8050 1950 60  0000 C CNN
-F 2 "" H 8050 1650 60  0001 C CNN
+F 2 "Housings_SOIC:SOIJ-8_5.3x5.3mm_Pitch1.27mm" H 8050 1650 60  0001 C CNN
 F 3 "" H 8050 1650 60  0001 C CNN
 	1    8050 1650
@@
 F 0 "SN1" H 6150 750 47  0000 C CNN
 F 1 "DS3232" H 6100 1950 47  0000 C CNN
-F 2 "" H 6150 1300 47  0001 C CNN
+F 2 "Housings_SOIC:SOIC-20W_7.5x12.8mm_Pitch1.27mm" H 6150 1300 47  0001 C CNN
 F 3 "" H 6150 1300 47  0001 C CNN
 	1    6150 1300
@@
 F 0 "U2" H 5700 3150 50  0000 C CNN
 F 1 "24LC256" H 6000 3150 50  0000 L CNN
-F 2 "Housings_SOIC:SOIC-8_3.9x4.9mm_Pitch1.27mm" H 6000 2650 50  0001 L CNN
+F 2 "Housings_DIP:DIP-8_W7.62mm_Socket" H 6000 2650 50  0001 L CNN
 F 3 "" H 5950 2800 50  0001 C CNN
 	1    5950 2900
@@
 F 0 "Q1" H 2000 4000 50  0000 L CNN
 F 1 "Q_NMOS_GSD" H 2000 3900 50  0000 L CNN
-F 2 "" H 2000 4050 50  0001 C CNN
+F 2 "TO_SOT_Packages_SMD:SOT-23_Handsoldering" H 2000 4050 50  0001 C CNN
 F 3 "" H 1800 3950 50  0001 C CNN
 	1    1800 3950
@@
 F 0 "U6" H 3750 950 60  0000 C CNN
 F 1 "MAX6730A" H 3750 1450 60  0000 C CNN
-F 2 "" H 3750 1200 60  0001 C CNN
+F 2 "TO_SOT_Packages_SMD:SOT-23-6_Handsoldering" H 3750 1200 60  0001 C CNN
 F 3 "" H 3750 1200 60  0001 C CNN
 	1    3750 1200
@@
 F 0 "R5" V 8280 6250 50  0000 C CNN
 F 1 "1k" V 8200 6250 50  0000 C CNN
-F 2 "" V 8130 6250 50  0001 C CNN
+F 2 "Resistors_SMD:R_0805_HandSoldering" V 8130 6250 50  0001 C CNN
 F 3 "" H 8200 6250 50  0001 C CNN
 	1    8200 6250
@@
 F 0 "R6" V 8280 6450 50  0000 C CNN
 F 1 "1k" V 8200 6450 50  0000 C CNN
-F 2 "" V 8130 6450 50  0001 C CNN
+F 2 "Resistors_SMD:R_0805_HandSoldering" V 8130 6450 50  0001 C CNN
 F 3 "" H 8200 6450 50  0001 C CNN
 	1    8200 6450
@@
 F 0 "U12" H 3900 2200 60  0000 C CNN
 F 1 "MS5540C" H 3900 2800 60  0000 C CNN
-F 2 "" H 3900 2500 60  0001 C CNN
+F 2 "aleksandr_footprints:MS5540C" H 3900 2500 60  0001 C CNN
 F 3 "" H 3900 2500 60  0001 C CNN
 	1    3900 2500
